File: ASTRA.kicad_pcb (KiCad board)
At the start: 2 copper layers, 36 parts, among them M1 NEMA17, M2 NEMA17, P1 12V-DC, SW1 TOP, SW2 BOTTOM, SW3 LEFT, SW4 RIGHT, SW5 SELECT, SW6 RETURN

Commit message: Ver 2
Parts:
- removed C7: 100nF, Capacitor_THT:C_Disc_D3.4mm_W2.1mm_P2.50mm
- removed R10: 8.2kR, Resistor_THT:R_Axial_DIN0207_L6.3mm_D2.5mm_P2.54mm_Vertical
- removed R11: 10kR, Resistor_THT:R_Axial_DIN0207_L6.3mm_D2.5mm_P2.54mm_Vertical
- removed R6: 1kR, Resistor_THT:R_Axial_DIN0207_L6.3mm_D2.5mm_P2.54mm_Vertical
- removed R7: 2.2kR, Resistor_THT:R_Axial_DIN0207_L6.3mm_D2.5mm_P2.54mm_Vertical
- removed R8: 4.7kR, Resistor_THT:R_Axial_DIN0207_L6.3mm_D2.5mm_P2.54mm_Vertical
- removed R9: 7.5kR, Resistor_THT:R_Axial_DIN0207_L6.3mm_D2.5mm_P2.54mm_Vertical
- added G1: BNO085, Connector_PinSocket_2.54mm:PinSocket_1x09_P2.54mm_Vertical, F.Cu at (175.9, 124.4)
- added U1: MCP23017x-x-SP, Package_DIP:DIP-28_W7.62mm, F.Cu at (171.4, 59.6)
- D1: value LED_YELLOW -> LED_RED
- D2: value LED_BLUE -> LED_GREEN
- D4: value LED_GREEN -> LED_BLUE
- D5: value LED_RED -> LED_YELLOW
- MC2: footprint ASTRAfootprints:WROOM32D Footprint -> RF_Module:ESP32-C3-DevKitM-1
- P1: footprint Connector_BarrelJack:BarrelJack_CUI_PJ-102AH_Horizontal -> Connector_BarrelJack:BarrelJack_Horizontal
- moved M2 123.0 mm to (121.0, 159.1), turned to 180 degrees
- moved M1 119.6 mm to (153.3, 159.1), turned to 180 degrees
- moved SW1 85.8 mm to (189.3, 82.4), turned to 90 degrees
- moved C2 79.7 mm to (103.9, 137.7)
- moved SW2 77.7 mm to (189.3, 77.8), turned to 90 degrees
- moved C4 74.0 mm to (107.8, 128.4), turned to 180 degrees
- moved C1 70.6 mm to (140.2, 128.2), turned to 180 degrees
- moved SW3 69.7 mm to (189.3, 73.2), turned to 90 degrees
- moved T2 67.3 mm to (114.2, 116.8), turned to 90 degrees
- moved C3 62.3 mm to (136.4, 137.3)
- moved D5 62.3 mm to (158.3, 73.0)
- moved SW4 61.8 mm to (189.3, 68.6), turned to 90 degrees
- moved D3 58.9 mm to (158.3, 64.7)
- moved MC2 57.1 mm to (118.8, 59.6)
- moved D1 55.9 mm to (158.6, 56.9)
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Connections:
- C1 pad 1: /CS -> /AD0
- C2 pad 2: /CS -> /AD0
- C3 pad 2: /CS -> /AD0
- C4 pad 1: /CS -> Net-(T1-MOT_VCC)
- C4 pad 2: Net-(T1-MOT_VCC) -> /AD0
- D1 pad 1: /CS -> /AD0
- D2 pad 1: /CS -> /AD0
- D3 pad 1: /CS -> /AD0
- D4 pad 1: /CS -> /AD0
- D5 pad 1: /CS -> /AD0
- MC2 pad 10: /D21 -> /D27
- MC2 pad 11: /D32 -> /D14
- MC2 pad 12: /D19 -> /D12
- MC2 pad 13: /D33 -> /D13
- MC2 pad 14: /D18 -> /AD0
- MC2 pad 15: /D25 -> unconnected-(MC2-Pin_29-Pad15)
- MC2 pad 16: /D5 -> /3V3
- MC2 pad 17: /D26 -> /AD0
- MC2 pad 18: /D17 -> /BL
- MC2 pad 19: /D27 -> /D2
- MC2 pad 2: /D23 -> unconnected-(MC2-Pin_3-Pad2)
- MC2 pad 20: /D16 -> /D4
- MC2 pad 21: /D14 -> /D16
- MC2 pad 22: /D4 -> /D17
- MC2 pad 23: /D12 -> /D5
- MC2 pad 24: /D2 -> /D18
- MC2 pad 25: /D13 -> /D16
- MC2 pad 26: /BL -> /D21
- MC2 pad 27: /CS -> /RX0/D3
- MC2 pad 28: /CS -> /TX0/D1
- MC2 pad 29: unconnected-(MC2-Pin_29-Pad29) -> /D22
- MC2 pad 30: /3V3 -> /D23
- MC2 pad 4: /D22 -> unconnected-(MC2-Pin_7-Pad4)
- MC2 pad 6: /TX0/D1 -> /D32
- MC2 pad 7: /D34 -> /D33
- MC2 pad 8: /RX0/D3 -> /D25
- MC2 pad 9: unconnected-(MC2-Pin_9-Pad9) -> /D26
- P1 pad 2: /CS -> /AD0
- R1 pad 1: Net-(D5-A) -> Net-(D1-A)
- R1 pad 2: /D4 -> Net-(U1-GPB0)
- R2 pad 1: Net-(D4-A) -> Net-(D2-A)
- R2 pad 2: /D16 -> Net-(U1-GPB1)
- R3 pad 2: /D17 -> Net-(U1-GPB2)
- R4 pad 1: Net-(D2-A) -> Net-(D4-A)
- R4 pad 2: /D5 -> Net-(U1-GPB3)
- R5 pad 1: Net-(D1-A) -> Net-(D5-A)
- R5 pad 2: /D18 -> Net-(U1-GPB4)
- S1 pad 1: /CS -> /AD0
- S1 pad 4: /D19 -> /D16
- S1 pad 7: /CS -> /AD0
- SW1 pad 2: /D34 -> /AD0
- SW2 pad 2: /D34 -> /AD0
- SW3 pad 2: /D34 -> /AD0
- SW4 pad 2: /D34 -> /AD0
- SW5 pad 2: /D34 -> /AD0
- SW6 pad 2: /D34 -> /AD0
- T1 pad 1: /3V3 -> Net-(T1-MOT_VCC)
- T1 pad 10: (no net) -> unconnected-(T1-MS1-Pad10)
- T1 pad 11: (no net) -> unconnected-(T1-MS2-Pad11)
- T1 pad 12: (no net) -> unconnected-(T1-SPREAD-Pad12)
- T1 pad 13: (no net) -> /D22
- T1 pad 14: (no net) -> /D23
- T1 pad 15: (no net) -> /D25
- T1 pad 16: (no net) -> /D33
- T1 pad 17: (no net) -> unconnected-(T1-Pad17)
- T1 pad 18: (no net) -> unconnected-(T1-Pad18)
- T1 pad 2: (no net) -> /AD0
- T1 pad 3: (no net) -> Net-(M1-Pin_4)
- T1 pad 4: (no net) -> Net-(M1-Pin_3)
- T1 pad 5: (no net) -> Net-(M1-Pin_2)
- T1 pad 6: (no net) -> Net-(M1-Pin_1)
- T1 pad 7: (no net) -> /3V3
- T1 pad 8: (no net) -> Net-(T1-I/O_GND)
- T1 pad 9: (no net) -> /D32
- T2 pad 1: /3V3 -> Net-(T1-MOT_VCC)
- T2 pad 10: (no net) -> unconnected-(T2-MS1-Pad10)
- T2 pad 11: (no net) -> unconnected-(T2-MS2-Pad11)
- T2 pad 12: (no net) -> unconnected-(T2-SPREAD-Pad12)
- T2 pad 13: (no net) -> /RX0/D3
- T2 pad 14: (no net) -> /TX0/D1
- T2 pad 15: (no net) -> /D14
- T2 pad 16: (no net) -> /D27
- T2 pad 17: (no net) -> unconnected-(T2-Pad17)
- T2 pad 18: (no net) -> unconnected-(T2-Pad18)
- T2 pad 2: (no net) -> /AD0
- T2 pad 3: (no net) -> Net-(M2-Pin_4)
- T2 pad 4: (no net) -> Net-(M2-Pin_3)
- T2 pad 5: (no net) -> Net-(M2-Pin_2)
- T2 pad 6: (no net) -> Net-(M2-Pin_1)
- T2 pad 7: (no net) -> /3V3
- T2 pad 8: (no net) -> Net-(T2-I/O_GND)
- T2 pad 9: (no net) -> /D26
Routing:
- net /AD0: track 0.00 -> 84.0 mm
- net Net-(M1-Pin_4): track 0.00 -> 38.7 mm
- net Net-(M2-Pin_4): track 0.00 -> 38.7 mm
- net Net-(M2-Pin_1): track 0.00 -> 37.2 mm
- net Net-(M1-Pin_1): track 0.00 -> 37.0 mm
- net Net-(M1-Pin_3): track 0.00 -> 36.7 mm
- net Net-(M2-Pin_3): track 0.00 -> 36.7 mm
- net Net-(M2-Pin_2): track 0.00 -> 36.1 mm
- net Net-(M1-Pin_2): track 0.00 -> 36.0 mm
- net /D17: track 0.00 -> 32.9 mm
- net /D16: track 0.00 -> 32.9 mm
- net Net-(T1-MOT_VCC): track 0.00 -> 29.6 mm
- net Net-(U1-GPA5): track 0.00 -> 12.4 mm
- net Net-(U1-GPA0): track 0.00 -> 12.3 mm
- net Net-(U1-GPA4): track 0.00 -> 11.5 mm
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
Commit message: V3 schematic
Parts:
- added B1: XL4016E1 Buck Converter, TerminalBlock:TerminalBlock_MaiXu_MX126-5.0-04P_1x04_P5.00mm, F.Cu at (155.5, 67.2)
- added C7: 100nF, Capacitor_THT:C_Disc_D3.4mm_W2.1mm_P2.50mm, F.Cu at (108.1, 124.3)
- added C8: 100nF, Capacitor_THT:C_Disc_D3.4mm_W2.1mm_P2.50mm, F.Cu at (108.1, 128.0)
- added R6: 4.7kR, Resistor_THT:R_Axial_DIN0207_L6.3mm_D2.5mm_P2.54mm_Vertical, F.Cu at (176.1, 84.4)
- added R7: 4.7kR, Resistor_THT:R_Axial_DIN0207_L6.3mm_D2.5mm_P2.54mm_Vertical, F.Cu at (176.1, 88.5)
- added SW7: RESET, Connector_PinHeader_2.54mm:PinHeader_1x02_P2.54mm_Vertical, F.Cu at (170.6, 123.4)
- C1: value 100nF -> 680uF; footprint Capacitor_THT:C_Disc_D3.4mm_W2.1mm_P2.50mm -> Capacitor_THT:CP_Radial_D8.0mm_P5.00mm
- C2: value 680uF -> 100nF; footprint Capacitor_THT:CP_Radial_D8.0mm_P5.00mm -> Capacitor_THT:C_Disc_D3.4mm_W2.1mm_P2.50mm
- MC2: value ~ -> ESP32
- S1: value ~ -> LCD Display ST7735S
- T1, T2: value ~ -> TMC2209
- moved P1 88.2 mm to (126.7, 132.3)
- moved M1 81.9 mm to (155.5, 77.3), turned to 0 degrees
- moved M2 79.6 mm to (155.5, 87.4), turned to 0 degrees
- moved SW6 68.1 mm to (166.0, 123.4), turned to 0 degrees
- moved SW5 65.6 mm to (161.4, 123.4), turned to 0 degrees
- moved SW4 63.7 mm to (156.8, 123.4), turned to 0 degrees
- moved SW3 62.4 mm to (152.2, 123.4), turned to 0 degrees
- moved SW1 61.8 mm to (143.0, 123.4), turned to 0 degrees
- moved SW2 61.8 mm to (147.6, 123.4), turned to 0 degrees
- moved G1 60.3 mm to (182.5, 64.4)
- moved T2 53.2 mm to (166.9, 110.2), turned to 0 degrees
- moved S1 50.3 mm to (135.6, 101.8)
- moved C5 46.3 mm to (108.1, 117.0)
- moved D5 32.1 mm to (135.7, 95.8)
- moved C1 30.0 mm to (114.7, 112.7), turned to 0 degrees
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Connections:
- net /D13 renamed /SCK
- C1 pad 1: /AD0 -> +12V
- C1 pad 2: Net-(T1-MOT_VCC) -> +12V
- C2 pad 1: Net-(T1-MOT_VCC) -> +12V
- C2 pad 2: /AD0 -> +12V
- C3 pad 1: Net-(T1-MOT_VCC) -> +12V
- C3 pad 2: /AD0 -> +12V
- C4 pad 1: Net-(T1-MOT_VCC) -> +12V
- C4 pad 2: /AD0 -> +12V
- C5 pad 1: /3V3 -> +3.3V
- C5 pad 2: Net-(T1-I/O_GND) -> +12V
- C6 pad 1: /3V3 -> +3.3V
- C6 pad 2: Net-(T2-I/O_GND) -> +12V
- D1 pad 1: /AD0 -> +12V
- D2 pad 1: /AD0 -> +12V
- D3 pad 1: /AD0 -> +12V
- D4 pad 1: /AD0 -> +12V
- D5 pad 1: /AD0 -> +12V
- G1 pad 1: /3V3 -> +3.3V
- G1 pad 2: /AD0 -> +12V
- G1 pad 3: /D17 -> /SCL
- G1 pad 4: /D16 -> /SDA
- G1 pad 5: /AD0 -> +12V
- G1 pad 6: unconnected-(G1-Pin_6-Pad6) -> +12V
- G1 pad 7: unconnected-(G1-Pin_7-Pad7) -> /INT
- G1 pad 8: unconnected-(G1-Pin_8-Pad8) -> +3.3V
- G1 pad 9: unconnected-(G1-Pin_9-Pad9) -> +12V
- MC2 pad 1: unconnected-(MC2-Pin_1-Pad1) -> Net-(MC2-Pin_1)
- MC2 pad 10: /D27 -> /RES
- MC2 pad 11: /D14 -> /MOSI
- MC2 pad 12: /D12 -> unconnected-(MC2-Pin_23-Pad12)
- MC2 pad 14: /AD0 -> +12V
- MC2 pad 16: /3V3 -> +3.3V
- MC2 pad 17: /AD0 -> +12V
- MC2 pad 18: /BL -> unconnected-(MC2-Pin_26-Pad18)
- MC2 pad 19: /D2 -> unconnected-(MC2-Pin_24-Pad19)
- MC2 pad 20: /D4 -> unconnected-(MC2-Pin_22-Pad20)
- MC2 pad 21: /D16 -> Net-(MC2-Pin_20)
- MC2 pad 22: /D17 -> Net-(MC2-Pin_18)
- MC2 pad 23: /D5 -> Net-(MC2-Pin_16)
- MC2 pad 24: /D18 -> Net-(MC2-Pin_14)
- MC2 pad 25: /D16 -> Net-(MC2-Pin_12)
- MC2 pad 26: /D21 -> Net-(MC2-Pin_10)
- MC2 pad 27: /RX0/D3 -> Net-(MC2-Pin_8)
- MC2 pad 28: /TX0/D1 -> Net-(MC2-Pin_6)
- MC2 pad 29: /D22 -> Net-(MC2-Pin_4)
- MC2 pad 30: /D23 -> Net-(MC2-Pin_2)
- MC2 pad 4: unconnected-(MC2-Pin_7-Pad4) -> /T2_DIAG
- MC2 pad 5: unconnected-(MC2-Pad5) -> /T1_DIAG
- MC2 pad 6: /D32 -> /SDA
- MC2 pad 7: /D33 -> /SCL
- MC2 pad 8: /D25 -> /BL
- MC2 pad 9: /D26 -> /DC
- P1 pad 1: Net-(T1-MOT_VCC) -> +12V
- P1 pad 2: /AD0 -> +12V
- R1 pad 2: Net-(U1-GPB0) -> Net-(U1-GPA0)
- R2 pad 2: Net-(U1-GPB1) -> Net-(U1-GPA1)
- R3 pad 2: Net-(U1-GPB2) -> Net-(U1-GPA2)
- R4 pad 2: Net-(U1-GPB3) -> Net-(U1-GPA3)
- R5 pad 2: Net-(U1-GPB4) -> Net-(U1-GPA4)
- S1 pad 1: /AD0 -> +12V
- S1 pad 2: /3V3 -> +3.3V
- S1 pad 4: /D16 -> /MOSI
- S1 pad 5: /D12 -> /RES
- S1 pad 6: /D21 -> /DC
- S1 pad 7: /AD0 -> +12V
- SW1 pad 1: Net-(U1-GPA0) -> Net-(U1-GPB0)
- SW1 pad 2: /AD0 -> +12V
- SW2 pad 1: Net-(U1-GPA1) -> Net-(U1-GPB1)
- SW2 pad 2: /AD0 -> +12V
- SW3 pad 1: Net-(U1-GPA2) -> Net-(U1-GPB2)
- SW3 pad 2: /AD0 -> +12V
- SW4 pad 1: Net-(U1-GPA3) -> Net-(U1-GPB3)
- SW4 pad 2: /AD0 -> +12V
- SW5 pad 1: Net-(U1-GPA4) -> Net-(U1-GPB4)
- SW5 pad 2: /AD0 -> +12V
- SW6 pad 1: Net-(U1-GPA5) -> Net-(U1-GPB5)
- SW6 pad 2: /AD0 -> +12V
- T1 pad 1: Net-(T1-MOT_VCC) -> +12V
- T1 pad 10: unconnected-(T1-MS1-Pad10) -> Net-(MC2-Pin_14)
- T1 pad 11: unconnected-(T1-MS2-Pad11) -> Net-(MC2-Pin_18)
- T1 pad 12: unconnected-(T1-SPREAD-Pad12) -> Net-(MC2-Pin_20)
- T1 pad 13: /D22 -> unconnected-(T1-SPRD-Pad13)
- T1 pad 14: /D23 -> unconnected-(T1-MS2-Pad14)
- T1 pad 15: /D25 -> unconnected-(T1-MS1-Pad15)
- T1 pad 16: /D33 -> Net-(MC2-Pin_12)
- T1 pad 18: unconnected-(T1-Pad18) -> /T1_DIAG
- T1 pad 2: /AD0 -> +3.3V
- T1 pad 3: Net-(M1-Pin_4) -> Net-(M1-Pin_3)
- T1 pad 4: Net-(M1-Pin_3) -> Net-(M1-Pin_1)
- T1 pad 6: Net-(M1-Pin_1) -> Net-(M1-Pin_4)
- T1 pad 7: /3V3 -> +12V
- T1 pad 8: Net-(T1-I/O_GND) -> +12V
- T1 pad 9: /D32 -> Net-(MC2-Pin_16)
- T2 pad 1: Net-(T1-MOT_VCC) -> +12V
- T2 pad 10: unconnected-(T2-MS1-Pad10) -> Net-(MC2-Pin_4)
- T2 pad 11: unconnected-(T2-MS2-Pad11) -> Net-(MC2-Pin_8)
- T2 pad 12: unconnected-(T2-SPREAD-Pad12) -> Net-(MC2-Pin_10)
- T2 pad 13: /RX0/D3 -> unconnected-(T2-SPRD-Pad13)
- T2 pad 14: /TX0/D1 -> unconnected-(T2-MS2-Pad14)
- T2 pad 15: /D14 -> unconnected-(T2-MS1-Pad15)
- T2 pad 16: /D27 -> Net-(MC2-Pin_2)
- T2 pad 18: unconnected-(T2-Pad18) -> /T2_DIAG
- T2 pad 2: /AD0 -> +3.3V
- T2 pad 3: Net-(M2-Pin_4) -> Net-(M2-Pin_3)
- T2 pad 4: Net-(M2-Pin_3) -> Net-(M2-Pin_1)
- T2 pad 6: Net-(M2-Pin_1) -> Net-(M2-Pin_4)
- T2 pad 7: /3V3 -> +12V
- T2 pad 8: Net-(T2-I/O_GND) -> +12V
- T2 pad 9: /D26 -> Net-(MC2-Pin_6)
- U1 pad 10: unconnected-(U1-V_{SS}-Pad10) -> +12V
- U1 pad 12: /D17 -> Net-(U1-SCK)
- U1 pad 13: /D16 -> Net-(U1-SDA)
- U1 pad 15: /AD0 -> +12V
- U1 pad 16: /AD0 -> +12V
- U1 pad 17: /AD0 -> +12V
- U1 pad 26: Net-(U1-GPA5) -> unconnected-(U1-GPA5-Pad26)
- U1 pad 6: unconnected-(U1-GPB5-Pad6) -> Net-(U1-GPB5)
- U1 pad 9: unconnected-(U1-V_{DD}-Pad9) -> +3.3V
Routing:
- net /AD0: track 84.0 -> 0.00 mm
- net Net-(M1-Pin_4): track 38.7 -> 0.00 mm
- net Net-(M2-Pin_4): track 38.7 -> 0.00 mm
- net Net-(M2-Pin_1): track 37.2 -> 0.00 mm
- net Net-(M1-Pin_1): track 37.0 -> 0.00 mm
- net Net-(M1-Pin_3): track 36.7 -> 0.00 mm
- net Net-(M2-Pin_3): track 36.7 -> 0.00 mm
- net Net-(M2-Pin_2): track 36.1 -> 0.00 mm
- net Net-(M1-Pin_2): track 36.0 -> 0.00 mm
- net /D17: track 32.9 -> 0.00 mm
- net /D16: track 32.9 -> 0.00 mm
- net Net-(T1-MOT_VCC): track 29.6 -> 0.00 mm
- net Net-(U1-GPA5): track 12.4 -> 0.00 mm
- net Net-(U1-GPA0): track 12.3 -> 0.00 mm
- net Net-(U1-GPA4): track 11.5 -> 0.00 mm
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Other:
- board outline added: 98.5 x 87.4 mm

Commit message: V3 finished schem
Parts:
- removed C8: 100nF, Capacitor_THT:C_Disc_D3.4mm_W2.1mm_P2.50mm
- removed G1: BNO085, Connector_PinSocket_2.54mm:PinSocket_1x09_P2.54mm_Vertical
- removed M1, M2: NEMA17, TerminalBlock:TerminalBlock_MaiXu_MX126-5.0-04P_1x04_P5.00mm
- removed R6, R7: 4.7kR, Resistor_THT:R_Axial_DIN0207_L6.3mm_D2.5mm_P2.54mm_Vertical
- added J1: RJ45 (NEMA 17), Connector_RJ:RJ45_Amphenol_54602-x08_Horizontal, F.Cu at (88.0, 55.1)
- added J2: RJ45 (NEMA 17), Connector_RJ:RJ45_Amphenol_54602-x08_Horizontal, F.Cu at (88.0, 71.5)
- added J3: RJ45 (BNO085), Connector_RJ:RJ45_Amphenol_54602-x08_Horizontal, F.Cu at (88.0, 128.8)
- B1: footprint TerminalBlock:TerminalBlock_MaiXu_MX126-5.0-04P_1x04_P5.00mm -> Connector_PinSocket_2.54mm:PinSocket_1x04_P2.54mm_Vertical
- C3: value 680uF -> 100nF; footprint Capacitor_THT:CP_Radial_D8.0mm_P5.00mm -> Capacitor_THT:C_Disc_D3.4mm_W2.1mm_P2.50mm
- MC2: footprint RF_Module:ESP32-C3-DevKitM-1 -> ASTRAfootprints:ESP32-WROOM-32D-Devkit
- P1: footprint Connector_BarrelJack:BarrelJack_Horizontal -> Connector_PinSocket_2.54mm:PinSocket_1x03_P2.54mm_Vertical
- moved T2 83.2 mm to (84.0, 117.1), turned to -90 degrees
- moved R1 76.6 mm to (114.0, 109.1), turned to 180 degrees
- moved R2 76.0 mm to (114.1, 112.1), turned to 180 degrees
- moved SW7 75.4 mm to (98.1, 102.8)
- moved R4 74.9 mm to (114.0, 118.2), turned to 180 degrees
- moved R5 71.2 mm to (114.0, 115.2), turned to 180 degrees
- moved R3 70.6 mm to (114.0, 106.0), turned to 180 degrees
- moved U1 70.2 mm to (127.0, 132.7), turned to -90 degrees
- moved B1 69.8 mm to (101.6, 111.5)
- moved T1 66.6 mm to (84.0, 98.6), turned to -90 degrees
- moved SW6 57.3 mm to (108.7, 123.1), turned to -90 degrees
- moved SW5 52.9 mm to (108.6, 119.6), turned to -90 degrees
- moved SW4 48.7 mm to (108.7, 116.0), turned to -90 degrees
- moved D1 48.1 mm to (117.5, 110.4)
- moved D2 48.1 mm to (117.5, 117.9)
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Connections:
- B1 pad 2: +12V -> GND
- B1 pad 3: +12V -> +5V
- B1 pad 4: +12V -> GND
- C1 pad 2: +12V -> GND
- C2 pad 2: +12V -> GND
- C3 pad 1: +12V -> +3.3V
- C3 pad 2: +12V -> GND
- C4 pad 2: +12V -> GND
- C5 pad 2: +12V -> GND
- C6 pad 2: +12V -> GND
- C7 pad 1: +3.3V -> Net-(C7-Pad1)
- C7 pad 2: +12V -> Net-(MC2-Pin_30)
- D1 pad 1: +12V -> GND
- D2 pad 1: +12V -> GND
- D3 pad 1: +12V -> GND
- D4 pad 1: +12V -> GND
- D5 pad 1: +12V -> GND
- MC2 pad 1: Net-(MC2-Pin_1) -> +3.3V
- MC2 pad 10: /RES -> /2EN
- MC2 pad 11: /MOSI -> /1DIR
- MC2 pad 12: unconnected-(MC2-Pin_23-Pad12) -> /1STEP
- MC2 pad 13: /SCK -> /1PDN
- MC2 pad 14: +12V -> /1UART
- MC2 pad 15: unconnected-(MC2-Pin_29-Pad15) -> /1EN
- MC2 pad 16: +3.3V -> Net-(MC2-Pin_30)
- MC2 pad 17: +12V -> unconnected-(MC2-Pin_28-Pad17)
- MC2 pad 19: unconnected-(MC2-Pin_24-Pad19) -> /T2_DIAG
- MC2 pad 2: unconnected-(MC2-Pin_3-Pad2) -> GND
- MC2 pad 20: unconnected-(MC2-Pin_22-Pad20) -> /T1_DIAG
- MC2 pad 21: Net-(MC2-Pin_20) -> /SDA
- MC2 pad 22: Net-(MC2-Pin_18) -> /SCL
- MC2 pad 23: Net-(MC2-Pin_16) -> /SCK
- MC2 pad 24: Net-(MC2-Pin_14) -> /MOSI
- MC2 pad 25: Net-(MC2-Pin_12) -> /RES
- MC2 pad 26: Net-(MC2-Pin_10) -> /DC
- MC2 pad 27: Net-(MC2-Pin_8) -> unconnected-(MC2-Pin_8-Pad27)
- MC2 pad 28: Net-(MC2-Pin_6) -> /BL
- MC2 pad 29: Net-(MC2-Pin_4) -> GND
- MC2 pad 3: unconnected-(MC2-Pin_5-Pad3) -> /2DIR
- MC2 pad 30: Net-(MC2-Pin_2) -> unconnected-(MC2-Pin_2-Pad30)
- MC2 pad 4: /T2_DIAG -> unconnected-(MC2-Pin_7-Pad4)
- MC2 pad 5: /T1_DIAG -> unconnected-(MC2-Pad5)
- MC2 pad 6: /SDA -> /2STEP
- MC2 pad 7: /SCL -> /2PDN
- MC2 pad 8: /BL -> unconnected-(MC2-Pin_15-Pad8)
- MC2 pad 9: /DC -> /2UART
- P1 pad 1: +12V -> GND
- R1 pad 2: Net-(U1-GPA0) -> Net-(U1-GPB0)
- R2 pad 2: Net-(U1-GPA1) -> Net-(U1-GPB1)
- R3 pad 2: Net-(U1-GPA2) -> Net-(U1-GPB2)
- R4 pad 2: Net-(U1-GPA3) -> Net-(U1-GPB3)
- R5 pad 2: Net-(U1-GPA4) -> Net-(U1-GPB4)
- S1 pad 1: +12V -> GND
- S1 pad 7: +12V -> GND
- SW1 pad 1: Net-(U1-GPB0) -> Net-(U1-GPA5)
- SW1 pad 2: +12V -> GND
- SW2 pad 1: Net-(U1-GPB1) -> Net-(U1-GPA4)
- SW2 pad 2: +12V -> GND
- SW3 pad 1: Net-(U1-GPB2) -> Net-(U1-GPA3)
- SW3 pad 2: +12V -> GND
- SW4 pad 1: Net-(U1-GPB3) -> Net-(U1-GPA2)
- SW4 pad 2: +12V -> GND
- SW5 pad 1: Net-(U1-GPB4) -> Net-(U1-GPA1)
- SW5 pad 2: +12V -> GND
- SW6 pad 1: Net-(U1-GPB5) -> Net-(U1-GPA0)
- SW6 pad 2: +12V -> GND
- SW7 pad 1: unconnected-(SW7-Pad1) -> GND
- SW7 pad 2: Net-(C8-Pad1) -> Net-(C7-Pad1)
- T1 pad 1: +12V -> GND
- T1 pad 10: Net-(MC2-Pin_14) -> /2STEP
- T1 pad 11: Net-(MC2-Pin_18) -> /2PDN
- T1 pad 12: Net-(MC2-Pin_20) -> /2UART
- T1 pad 16: Net-(MC2-Pin_12) -> /2EN
- T1 pad 7: +12V -> GND
- T1 pad 9: Net-(MC2-Pin_16) -> /2DIR
- T2 pad 1: +12V -> GND
- T2 pad 10: Net-(MC2-Pin_4) -> /1STEP
- T2 pad 11: Net-(MC2-Pin_8) -> /1PDN
- T2 pad 12: Net-(MC2-Pin_10) -> /1UART
- T2 pad 16: Net-(MC2-Pin_2) -> /1EN
- T2 pad 7: +12V -> GND
- T2 pad 9: Net-(MC2-Pin_6) -> /1DIR
- U1 pad 10: +12V -> GND
- U1 pad 12: Net-(U1-SCK) -> /SCL
- U1 pad 13: Net-(U1-SDA) -> /SDA
- U1 pad 15: +12V -> GND
- U1 pad 16: +12V -> GND
- U1 pad 17: +12V -> GND
- U1 pad 26: unconnected-(U1-GPA5-Pad26) -> Net-(U1-GPA5)
- U1 pad 6: Net-(U1-GPB5) -> unconnected-(U1-GPB5-Pad6)
Routing:
- net GND: track 0.00 -> 273.8 mm, vias 0 -> 4
- net /T1_DIAG: track 0.00 -> 107.6 mm
- net +3.3V: track 0.00 -> 105.5 mm, vias 0 -> 3
- net /2UART: track 0.00 -> 98.8 mm
- net /2EN: track 0.00 -> 95.5 mm
- net +12V: track 0.00 -> 87.2 mm, vias 0 -> 1
- net /BL: track 0.00 -> 86.3 mm
- net /T2_DIAG: track 0.00 -> 80.7 mm
- net /SCL: track 0.00 -> 77.9 mm, vias 0 -> 1
- net /SDA: track 0.00 -> 71.3 mm, vias 0 -> 1
- net /2PDN: track 0.00 -> 53.4 mm, vias 0 -> 2
- net /1EN: track 0.00 -> 51.1 mm
- net /2STEP: track 0.00 -> 46.4 mm
- net Net-(T2-M1B): track 0.00 -> 46.3 mm
- net /1DIR: track 0.00 -> 43.7 mm
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Other:
- board size 98.5 x 87.4 mm -> 57 x 92 mm
