File: ASTRA.kicad_sch (KiCad schematic)
At the start: 36 parts, among them M1 NEMA17, M2 NEMA17, P1 12V-DC, SW1 TOP, SW2 BOTTOM, SW3 LEFT, SW4 RIGHT, SW5 SELECT, SW6 RETURN

Commit message: Ver 2
Parts:
- removed C7: 100nF, Capacitor_THT:C_Disc_D3.4mm_W2.1mm_P2.50mm, symbol Device:C
- removed R10: 8.2kR, Resistor_THT:R_Axial_DIN0207_L6.3mm_D2.5mm_P2.54mm_Vertical, symbol Device:R
- removed R11: 10kR, Resistor_THT:R_Axial_DIN0207_L6.3mm_D2.5mm_P2.54mm_Vertical, symbol Device:R
- removed R6: 1kR, Resistor_THT:R_Axial_DIN0207_L6.3mm_D2.5mm_P2.54mm_Vertical, symbol Device:R
- removed R7: 2.2kR, Resistor_THT:R_Axial_DIN0207_L6.3mm_D2.5mm_P2.54mm_Vertical, symbol Device:R
- removed R8: 4.7kR, Resistor_THT:R_Axial_DIN0207_L6.3mm_D2.5mm_P2.54mm_Vertical, symbol Device:R
- removed R9: 7.5kR, Resistor_THT:R_Axial_DIN0207_L6.3mm_D2.5mm_P2.54mm_Vertical, symbol Device:R
- added G1: BNO085, Connector_PinSocket_2.54mm:PinSocket_1x09_P2.54mm_Vertical, symbol Connector_Generic:Conn_01x09
- added U1: MCP23017x-x-SP, Package_DIP:DIP-28_W7.62mm, symbol Interface_Expansion:MCP23017x-x-SP
- MC2: footprint ASTRAfootprints:WROOM32D Footprint -> RF_Module:ESP32-C3-DevKitM-1
- P1: footprint Connector_BarrelJack:BarrelJack_CUI_PJ-102AH_Horizontal -> Connector_BarrelJack:BarrelJack_Horizontal
- renumbered D5 to D1, D4 to D2, D2 to D4, D1 to D5
Connections:
- net 3V3: now also MC2.16 (Pin_30), T1.7 (I/O_VCC), T2.7 (I/O_VCC), G1.1 (Pin_1); no longer MC2.30 (Pin_30), T1.1 (STEP), T2.1 (STEP)
- net BL: now also MC2.18 (Pin_26); no longer MC2.26 (Pin_26)
- net D12: now also MC2.12 (Pin_23); no longer MC2.23 (Pin_23)
- net D13: now also MC2.13 (Pin_25); no longer MC2.25 (Pin_25)
- net D14: now also MC2.11 (Pin_21), T2.15 (DIR); no longer MC2.21 (Pin_21), T2.1 (STEP)
- net D16: now also MC2.21 (Pin_20), MC2.25 (Pin_12), S1.4 (Pin_4), G1.4 (Pin_4), U1.13 (SDA); no longer MC2.20 (Pin_20), R2.2
- net D17: now also MC2.22 (Pin_18), G1.3 (Pin_3), U1.12 (SCK); no longer MC2.18 (Pin_18), R3.2
- net D18: now also MC2.24 (Pin_14); no longer MC2.14 (Pin_14), R5.2
- net D2: now also MC2.19 (Pin_24); no longer MC2.24 (Pin_24)
- net D21: now also MC2.26 (Pin_10); no longer MC2.10 (Pin_10)
- net D22: now also MC2.29 (Pin_4), T1.13 (PDN_UART); no longer MC2.4 (Pin_4), T1.1 (STEP)
- net D23: now also MC2.30 (Pin_2), T1.14 (PDN_UART); no longer MC2.2 (Pin_2), T1.1 (STEP)
- net D25: now also MC2.8 (Pin_15), T1.15 (DIR); no longer MC2.15 (Pin_15), T1.1 (STEP)
- net D26: now also MC2.9 (Pin_17), T2.9 (EN); no longer MC2.17 (Pin_17), T2.1 (STEP)
- net D27: now also MC2.10 (Pin_19), T2.16 (STEP); no longer MC2.19 (Pin_19), T2.1 (STEP)
- net D32: now also MC2.6 (Pin_11), T1.9 (EN); no longer MC2.11 (Pin_11), T1.1 (STEP)
- net D33: now also MC2.7 (Pin_13), T1.16 (STEP); no longer MC2.13 (Pin_13), T1.1 (STEP)
- net D34: no longer MC2.7 (Pin_7), SW1.2, SW2.2, SW3.2, SW4.2, SW5.2, SW6.2
- net D4: now also MC2.20 (Pin_22); no longer MC2.22 (Pin_22), R1.2
- net D5: now also MC2.23 (Pin_16); no longer MC2.16 (Pin_16), R4.2
- net RX0/D3: now also MC2.27 (Pin_8), T2.13 (PDN_UART); no longer MC2.8 (Pin_8), T2.1 (STEP)
- net TX0/D1: now also MC2.28 (Pin_6), T2.14 (PDN_UART); no longer MC2.6 (Pin_6), T2.1 (STEP)
- net at M2.1 (Pin_1): now also T2.6 (M1B); no longer T2.1 (STEP)
- net at M2.2 (Pin_2): now also T2.5 (M1A); no longer T2.1 (STEP)
- net at M2.3 (Pin_3): now also T2.4 (M2A); no longer T2.1 (STEP)
- net at M2.4 (Pin_4): now also T2.3 (M2B); no longer T2.1 (STEP)
- net at SW5.1: now also U1.25 (GPA4)
- net at SW1.1: now also U1.21 (GPA0)
- net at SW4.1: now also U1.24 (GPA3)
- net at SW6.1: now also U1.26 (GPA5)
- net at C1.2, C2.1, C3.1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: now also C4.1; no longer C4.2
- net at SW2.1: now also U1.22 (GPA1)
- net at SW3.1: now also U1.23 (GPA2)
- net at C6.2: now also T2.8 (I/O_GND); no longer T2.1 (STEP)
- net at C5.2: now also T1.8 (I/O_GND); no longer T1.1 (STEP)
- net at M1.1 (Pin_1): now also T1.6 (M1B); no longer T1.1 (STEP)
- net at M1.2 (Pin_2): now also T1.5 (M1A); no longer T1.1 (STEP)
- net at M1.3 (Pin_3): now also T1.4 (M2A); no longer T1.1 (STEP)
- net at M1.4 (Pin_4): now also T1.3 (M2B); no longer T1.1 (STEP)
- net CS renamed AD0
- net AD0: now also C4.2, MC2.14 (Pin_27), MC2.17 (Pin_28), SW1.2, SW2.2, SW3.2, SW4.2, SW5.2, SW6.2, T1.2 (MOT_GND), T2.2 (MOT_GND), G1.2 (Pin_2), G1.5 (Pin_5), U1.15 (A0), U1.16 (A1), U1.17 (A2); no longer C4.1, MC2.27 (Pin_27), MC2.28 (Pin_28), T1.1 (STEP), T2.1 (STEP)
- removed net D19: MC2.12 (Pin_12), S1.4 (Pin_4)
- new net: R2.2, U1.2 (GPB1)
- new net: R1.2, U1.1 (GPB0)
- new net: R5.2, U1.5 (GPB4)
- new net: R4.2, U1.4 (GPB3)
- new net: R3.2, U1.3 (GPB2)
Other:
- moved on the sheet: C4, D1, D2, D3, D4, D5, R1, R2, R3, R4, R5, S1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

Commit message: V3 schematic
Parts:
- removed M1, M2: NEMA17, TerminalBlock:TerminalBlock_MaiXu_MX126-5.0-04P_1x04_P5.00mm, symbol Connector_Generic:Conn_01x04
- removed T1, T2: (no value), ASTRAfootprints:TMC2209module, symbol ASTRAsymbols:TMC2209_Module
- added B1: XL4016E1 Buck Converter, TerminalBlock:TerminalBlock_MaiXu_MX126-5.0-04P_1x04_P5.00mm, symbol Connector_Generic:Conn_01x04
- added C7, C8: 100nF, Capacitor_THT:C_Disc_D3.4mm_W2.1mm_P2.50mm, symbol Device:C
- added J1, J2: RJ45 (NEMA 17), symbol Connector:RJ45
- added R6, R7: 4.7kR, Resistor_THT:R_Axial_DIN0207_L6.3mm_D2.5mm_P2.54mm_Vertical, symbol Device:R
- added SW7: RESET, Connector_PinHeader_2.54mm:PinHeader_1x02_P2.54mm_Vertical, symbol Switch:SW_Push
- added T1, T2: TMC2209, ASTRAfootprints:TMC2209module, symbol ASTRAsymbols:TMC2209_SILENTSTEPSTICK
- MC2: value (none) -> ESP32
- S1: value (none) -> LCD Display ST7735S
- renumbered C2 to C1, C1 to C2
Connections:
- net AD0 is gone; now on net +12V: C1.2, C2.1, C3.2, C4.2, D1.1 (K), D2.1 (K), D3.1 (K), D4.1 (K), D5.1 (K), G1.2 (Pin_2), G1.5 (Pin_5), MC2.14 (Pin_27), MC2.17 (Pin_28), P1.2, S1.1 (Pin_1), S1.7 (Pin_7), SW1.2, SW2.2, SW3.2, SW4.2, SW5.2, SW6.2, U1.15 (A0), U1.16 (A1), U1.17 (A2)
- net 3V3: no longer C5.1, C6.1, G1.1 (Pin_1), MC2.16 (Pin_30), S1.2 (Pin_2)
- net BL: now also MC2.8 (Pin_15); no longer MC2.18 (Pin_26)
- net D12: no longer MC2.12 (Pin_23), S1.5 (Pin_5)
- net D13: no longer MC2.13 (Pin_25), S1.3 (Pin_3)
- net D14: no longer MC2.11 (Pin_21)
- net D16: no longer G1.4 (Pin_4), MC2.21 (Pin_20), MC2.25 (Pin_12), S1.4 (Pin_4), U1.13 (SDA)
- net D17: no longer G1.3 (Pin_3), MC2.22 (Pin_18), U1.12 (SCK)
- net D18: no longer MC2.24 (Pin_14)
- net D2: no longer MC2.19 (Pin_24)
- net D21: no longer MC2.26 (Pin_10), S1.6 (Pin_6)
- net D22: no longer MC2.29 (Pin_4)
- net D23: no longer MC2.30 (Pin_2)
- net D25: no longer MC2.8 (Pin_15)
- net D26: no longer MC2.9 (Pin_17)
- net D27: no longer MC2.10 (Pin_19)
- net D32: no longer MC2.6 (Pin_11)
- net D33: no longer MC2.7 (Pin_13)
- net D4: no longer MC2.20 (Pin_22)
- net D5: no longer MC2.23 (Pin_16)
- net INT: now also G1.7 (Pin_7)
- net RX0/D3: no longer MC2.27 (Pin_8)
- net TX0/D1: no longer MC2.28 (Pin_6)
- net at SW5.1: now also U1.5 (GPB4); no longer U1.25 (GPA4)
- net at SW4.1: now also U1.4 (GPB3); no longer U1.24 (GPA3)
- net at R2.2: now also U1.22 (GPA1); no longer U1.2 (GPB1)
- net at MC2.1 (Pin_1): now also C8.2
- net T2_DIAG: now reaches MC2.4 (Pin_7)
- net T2_DIAG: now also T2.18 (DIAG)
- net T1_DIAG: now reaches MC2.5
- net T1_DIAG: now also T1.18 (DIAG)
- net at R1.2: now also U1.21 (GPA0); no longer U1.1 (GPB0)
- net +12V: now reaches C1.1, C2.2, C3.1, C4.1, P1.1
- net +12V: now also C5.2, C6.2, G1.6 (Pin_6), G1.9 (Pin_9), U1.10 (V_{SS}), B1.1 (Pin_1), B1.2 (Pin_2), B1.3 (Pin_3), B1.4 (Pin_4), C7.2, T1.1 (GND), T1.7 (GND), T1.8 (VM), T2.1 (GND), T2.7 (GND), T2.8 (VM)
- net at R5.2: now also U1.25 (GPA4); no longer U1.5 (GPB4)
- net at R4.2: now also U1.24 (GPA3); no longer U1.4 (GPB3)
- net at U1.23 (GPA2): now also R3.2; no longer SW3.1
- net at SW2.1: now also U1.2 (GPB1); no longer U1.22 (GPA1)
- net at U1.3 (GPB2): now also SW3.1; no longer R3.2
- net at SW1.1: now also U1.1 (GPB0); no longer U1.21 (GPA0)
- net at U1.26 (GPA5): no longer SW6.1
- net at U1.6 (GPB5): now also SW6.1
- net +3.3V: now reaches U1.9 (V_{DD})
- net +3.3V: now also C5.1, C6.1, G1.1 (Pin_1), G1.8 (Pin_8), MC2.16 (Pin_30), S1.2 (Pin_2), C7.1, T1.2 (VIO), T2.2 (VIO)
- new net: MC2.21 (Pin_20), T1.12 (UART)
- new net: MC2.22 (Pin_18), T1.11 (PDN)
- new net: MC2.23 (Pin_16), T1.9 (DIR)
- new net: MC2.24 (Pin_14), T1.10 (STEP)
- new net: MC2.25 (Pin_12), T1.16 (~{EN})
- new net: MC2.26 (Pin_10), T2.12 (UART)
- new net: MC2.27 (Pin_8), T2.11 (PDN)
- new net: MC2.28 (Pin_6), T2.9 (DIR)
- new net: MC2.29 (Pin_4), T2.10 (STEP)
- new net: MC2.30 (Pin_2), T2.16 (~{EN})
- new net: J1.5, J1.6, T1.3 (M1B)
- new net: J1.1, J1.2, T1.4 (M1A)
- new net: J1.3, J1.4, T1.5 (M2A)
- new net: J1.7, J1.8, T1.6 (M2B)
- new net: R6.2, U1.12 (SCK)
- new net: R7.2, U1.13 (SDA)
- new net: C8.1, SW7.2
- new net: J2.1, J2.2, T2.4 (M1A)
- new net: J2.3, J2.4, T2.5 (M2A)
- new net: J2.5, J2.6, T2.3 (M1B)
- new net: J2.7, J2.8, T2.6 (M2B)
- new net DC: MC2.9 (Pin_17), S1.6 (Pin_6)
- new net MOSI: MC2.11 (Pin_21), S1.4 (Pin_4)
- new net RES: MC2.10 (Pin_19), S1.5 (Pin_5)
- new net SCK: MC2.13 (Pin_25), S1.3 (Pin_3)
- new net SCL: G1.3 (Pin_3), MC2.7 (Pin_13), R6.1
- new net SDA: G1.4 (Pin_4), MC2.6 (Pin_11), R7.1
Other:
- moved on the sheet: C1, C2, D1, D2, D3, D4, D5, R1, R2, R3, R4, R5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

Commit message: V3 finished schem
Parts:
- removed C1: 680uF, Capacitor_THT:CP_Radial_D8.0mm_P5.00mm, symbol Device:C_Polarized
- removed C8: 100nF, Capacitor_THT:C_Disc_D3.4mm_W2.1mm_P2.50mm, symbol Device:C
- removed R6, R7: 4.7kR, Resistor_THT:R_Axial_DIN0207_L6.3mm_D2.5mm_P2.54mm_Vertical, symbol Device:R
- added C7: 100nF, Capacitor_THT:C_Disc_D3.4mm_W2.1mm_P2.50mm, symbol Device:C
- added J3, J4: RJ45 (BNO085), Connector_RJ:RJ45_Amphenol_54602-x08_Horizontal, symbol Connector:RJ45
- B1: footprint TerminalBlock:TerminalBlock_MaiXu_MX126-5.0-04P_1x04_P5.00mm -> Connector_PinSocket_2.54mm:PinSocket_1x04_P2.54mm_Vertical
- J1, J2: footprint (none) -> Connector_RJ:RJ45_Amphenol_54602-x08_Horizontal
- MC2: footprint RF_Module:ESP32-C3-DevKitM-1 -> ASTRAfootprints:ESP32-WROOM-32D-Devkit
- P1: footprint Connector_BarrelJack:BarrelJack_Horizontal -> Connector_PinSocket_2.54mm:PinSocket_1x03_P2.54mm_Vertical
- renumbered C3 to C1, C4 to C2, C6 to C3, C2 to C4, C7 to C6
Connections:
- net +12V: no longer B1.2 (Pin_2), B1.3 (Pin_3), B1.4 (Pin_4), C1.2, C2.2, C3.2, C4.2, C5.2, C6.2, D1.1 (K), D2.1 (K), D3.1 (K), D4.1 (K), D5.1 (K), G1.2 (Pin_2), G1.5 (Pin_5), G1.6 (Pin_6), G1.9 (Pin_9), MC2.14 (Pin_27), MC2.17 (Pin_28), P1.1, S1.1 (Pin_1), S1.7 (Pin_7), SW1.2, SW2.2, SW3.2, SW4.2, SW5.2, SW6.2, T1.1 (GND), T1.7 (GND), T2.1 (GND), T2.7 (GND), U1.10 (V_{SS}), U1.15 (A0), U1.16 (A1), U1.17 (A2)
- net +3.3V: now also MC2.1 (Pin_1), J3.6, J4.6; no longer MC2.16 (Pin_30)
- net BL: now also MC2.28 (Pin_6); no longer MC2.8 (Pin_15)
- net DC: now also MC2.26 (Pin_10); no longer MC2.9 (Pin_17)
- net MOSI: now also MC2.24 (Pin_14); no longer MC2.11 (Pin_21)
- net RES: now also MC2.25 (Pin_12); no longer MC2.10 (Pin_19)
- net SCK: now also MC2.23 (Pin_16); no longer MC2.13 (Pin_25)
- net SCL: now also MC2.22 (Pin_18), U1.12 (SCK), J3.2, J4.4; no longer MC2.7 (Pin_13)
- net SDA: now also MC2.21 (Pin_20), U1.13 (SDA), J3.4, J4.2; no longer MC2.6 (Pin_11)
- net T1_DIAG: now also MC2.20 (Pin_22); no longer MC2.5
- net T2_DIAG: now also MC2.19 (Pin_24); no longer MC2.4 (Pin_7)
- net at SW5.1: now also U1.22 (GPA1); no longer U1.5 (GPB4)
- net at SW4.1: now also U1.23 (GPA2); no longer U1.4 (GPB3)
- net at R2.2: now also U1.2 (GPB1); no longer U1.22 (GPA1)
- net 1STEP: now reaches MC2.12 (Pin_23)
- net 1STEP: now also T2.10 (STEP)
- net 1EN: now reaches MC2.15 (Pin_29)
- net 1EN: now also T2.16 (~{EN})
- net GND: now reaches MC2.2 (Pin_3)
- net GND: now also B1.2 (Pin_2), B1.4 (Pin_4), C1.2, C2.2, C3.2, C4.2, C5.2, C6.2, D1.1 (K), D2.1 (K), D3.1 (K), D4.1 (K), D5.1 (K), G1.2 (Pin_2), G1.5 (Pin_5), G1.6 (Pin_6), G1.9 (Pin_9), MC2.29 (Pin_4), P1.1, S1.1 (Pin_1), S1.7 (Pin_7), SW1.2, SW2.2, SW3.2, SW4.2, SW5.2, SW6.2, SW7.1, T1.1 (GND), T1.7 (GND), T2.1 (GND), T2.7 (GND), U1.10 (V_{SS}), U1.15 (A0), U1.16 (A1), U1.17 (A2), J3.1, J3.3, J3.5, J4.1, J4.3, J4.5
- net 2UART: now reaches T1.12 (UART)
- net 2UART: now also MC2.9 (Pin_17); no longer MC2.21 (Pin_20)
- net 2PDN: now reaches T1.11 (PDN)
- net 2PDN: now also MC2.7 (Pin_13); no longer MC2.22 (Pin_18)
- net 2DIR: now reaches T1.9 (DIR)
- net 2DIR: now also MC2.3 (Pin_5); no longer MC2.23 (Pin_16)
- net 2STEP: now reaches T1.10 (STEP)
- net 2STEP: now also MC2.6 (Pin_11); no longer MC2.24 (Pin_14)
- net 2EN: now reaches T1.16 (~{EN})
- net 2EN: now also MC2.10 (Pin_19); no longer MC2.25 (Pin_12)
- net 1UART: now reaches T2.12 (UART)
- net 1UART: now also MC2.14 (Pin_27); no longer MC2.26 (Pin_10)
- net at MC2.27 (Pin_8): no longer T2.11 (PDN)
- net 1DIR: now reaches T2.9 (DIR)
- net 1DIR: now also MC2.11 (Pin_21); no longer MC2.28 (Pin_6)
- net at MC2.30 (Pin_2): no longer T2.16 (~{EN})
- net at R1.2: now also U1.1 (GPB0); no longer U1.21 (GPA0)
- net at J1.5, J1.6: now also T1.5 (M2A); no longer T1.3 (M1B)
- net at J1.1, J1.2: now also T1.3 (M1B); no longer T1.4 (M1A)
- net at J1.3, J1.4: now also T1.4 (M1A); no longer T1.5 (M2A)
- net at U1.25 (GPA4): now also SW2.1; no longer R5.2
- net at SW1.1: now also U1.26 (GPA5); no longer U1.1 (GPB0)
- net at R3.2: now also U1.3 (GPB2); no longer U1.23 (GPA2)
- net at U1.24 (GPA3): now also SW3.1; no longer R4.2
- net at SW6.1: now also U1.21 (GPA0); no longer U1.6 (GPB5)
- net at SW7.2: now also C7.1
- net at J2.1, J2.2: now also T2.3 (M1B); no longer T2.4 (M1A)
- net at J2.3, J2.4: now also T2.4 (M1A); no longer T2.5 (M2A)
- net at J2.5, J2.6: now also T2.5 (M2A); no longer T2.3 (M1B)
- new net: C7.2, MC2.16 (Pin_30)
- new net: R4.2, U1.4 (GPB3)
- new net: R5.2, U1.5 (GPB4)
- new net +5V: B1.3 (Pin_3)
- new net 1PDN: MC2.13 (Pin_25), T2.11 (PDN)
Other:
- moved on the sheet: C4, G1, MC2
