File: AstraController/ASTRA.kicad_sch (KiCad schematic)
At the start: 36 parts, among them J1 RJ45 (NEMA 17), J2 RJ45 (NEMA 17), J3 RJ45 (BNO085), J4 RJ45 (BNO085), P1 12V-DC, SW1 TOP, SW2 BOTTOM, SW3 LEFT, SW4 RIGHT, SW5 SELECT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

Commit message: V4 hardware
Parts:
- added J5: USB_A, Connector_USB:USB_A_Connfly_DS1095, symbol Connector:USB_A
- C1: footprint Capacitor_THT:CP_Radial_D8.0mm_P5.00mm -> Capacitor_THT:CP_Radial_D10.0mm_P5.00mm
- C2, C3, C4, C5, C6, C7: footprint Capacitor_THT:C_Disc_D3.4mm_W2.1mm_P2.50mm -> Capacitor_SMD:C_0805_2012Metric_Pad1.18x1.45mm_HandSolder
- D1, D2, D3, D4, D5: footprint LED_THT:LED_D5.0mm -> LED_SMD:LED_0805_2012Metric_Pad1.15x1.40mm_HandSolder
- R1, R2, R3, R4, R5: footprint Resistor_THT:R_Axial_DIN0207_L6.3mm_D2.5mm_P2.54mm_Vertical -> Resistor_SMD:R_0805_2012Metric_Pad1.20x1.40mm_HandSolder
- SW1, SW2, SW3, SW4, SW5, SW6, SW7: footprint Connector_PinHeader_2.54mm:PinHeader_1x02_P2.54mm_Vertical -> Connector_PinSocket_2.54mm:PinSocket_1x02_P2.54mm_Vertical
Connections:
- net +5V: now also J5.1 (VBUS)
- net GND: now also J5.4 (GND), J5.SH (Shield)
- net LEFT: now reaches U1.3 (GPB2)
- net LEFT: now also SW3.1; no longer R3.2
- net RED: now reaches R1.2
- net RED: now also U1.4 (GPB3); no longer U1.1 (GPB0)
- net at U1.23 (GPA2): no longer SW4.1
- net BOTTOM: now reaches U1.2 (GPB1)
- net BOTTOM: now also SW2.1; no longer R2.2
- net at U1.21 (GPA0): no longer SW6.1
- net at U1.22 (GPA1): no longer SW5.1
- net at U1.24 (GPA3): no longer SW3.1
- net at U1.25 (GPA4): no longer SW2.1
- net RETURN: now reaches U1.26 (GPA5)
- net RETURN: now also SW6.1; no longer SW1.1
- net SELECT: now reaches U1.27 (GPA6)
- net SELECT: now also SW5.1
- net RIGHT: now reaches U1.28 (GPA7)
- net RIGHT: now also SW4.1
- net BLUE: now reaches R4.2
- net BLUE: now also U1.7 (GPB6); no longer U1.4 (GPB3)
- net GREEN: now reaches U1.5 (GPB4)
- net GREEN: now also R2.2; no longer R5.2
- net WHITE: now reaches U1.6 (GPB5)
- net WHITE: now also R3.2
- net YELLOW: now reaches U1.8 (GPB7)
- net YELLOW: now also R5.2
- new net TOP: SW1.1, U1.1 (GPB0)
Other:
- moved on the sheet: D1, D2, D3, D4, D5, R1, R2, R3, R4, R5, SW1, SW2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
