File: AstraController/ASTRA.kicad_pcb (KiCad board)
At the start: 4 copper layers, 55 x 85 mm, 35 parts, among them J1 RJ45 (NEMA 17), J2 RJ45 (NEMA 17), J3 RJ45 (BNO085), J5 USB_A, P1 12V-DC, SW1 TOP, SW2 BOTTOM, SW3 LEFT, SW4 RIGHT, SW5 SELECT, SW6 RETURN, SW7 RESET, T1 TMC2209, T2 TMC2209, U1 MCP23017x-x-SP

Commit message: idk
Parts:
- moved S1 52.6 mm to (157.9, 68.2), turned to 90 degrees
- moved P1 45.2 mm to (180.0, 110.9), turned to 90 degrees
- moved B1 44.6 mm to (178.2, 114.5), turned to 90 degrees
- moved D5 37.6 mm to (186.3, 61.2), turned to 180 degrees
- moved C6 36.5 mm to (175.2, 61.1), turned to 0 degrees
- moved R5 35.2 mm to (182.6, 61.2), turned to 180 degrees
- moved U1 34.4 mm to (153.7, 59.0), turned to 90 degrees
- moved D4 34.1 mm to (186.3, 63.1), turned to 180 degrees
- moved SW5 33.3 mm to (150.3, 52.1), turned to 0 degrees
- moved R4 31.4 mm to (182.6, 63.1), turned to 180 degrees
- moved SW1 31.1 mm to (153.9, 62.0), turned to 0 degrees
- moved D3 30.7 mm to (186.3, 65.1), turned to 180 degrees
- moved R3 27.7 mm to (182.6, 65.1), turned to 180 degrees
- moved D2 27.4 mm to (186.3, 67.0), turned to 180 degrees
- moved SW6 26.4 mm to (150.3, 58.2), turned to 0 degrees
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Connections:
- MC2 pad 19: /T2_DIAG -> /T1_DIAG
- MC2 pad 20: /T1_DIAG -> /T2_DIAG
- U1 pad 1: /TOP -> /RETURN
- U1 pad 2: /BOTTOM -> /TOP
- U1 pad 21: unconnected-(U1-GPA0-Pad21) -> /YELLOW
- U1 pad 22: unconnected-(U1-GPA1-Pad22) -> /BLUE
- U1 pad 26: /RETURN -> unconnected-(U1-GPA5-Pad26)
- U1 pad 27: /SELECT -> unconnected-(U1-GPA6-Pad27)
- U1 pad 28: /RIGHT -> /SELECT
- U1 pad 3: /LEFT -> /BOTTOM
- U1 pad 4: /RED -> /LEFT
- U1 pad 5: /GREEN -> /RIGHT
- U1 pad 6: /WHITE -> /RED
- U1 pad 7: /BLUE -> /GREEN
- U1 pad 8: /YELLOW -> /WHITE
Routing:
- net /BL: track 114.4 -> 4.29 mm
- net /DC: track 104.6 -> 4.29 mm
- net /RES: track 98.4 -> 4.29 mm
- net /MOSI: track 93.7 -> 4.29 mm
- net /T2_DIAG: track 127.5 -> 40.6 mm
- net /SCK: track 89.1 -> 4.29 mm
- net +5V: track 21.6 -> 101.9 mm
- net /1PDN: track 50.6 -> 13.3 mm
- net /1STEP: track 44.7 -> 13.3 mm
- net +12V: track 77.3 -> 46.9 mm
- net Net-(MC2-Pin_30): track 30.9 -> 3.20 mm
- net /RETURN: track 31.2 -> 3.68 mm
- net /2EN: track 40.9 -> 13.8 mm, vias 1 -> 0
- net /1EN: track 31.8 -> 5.64 mm
- net /SCL: track 77.3 -> 102.2 mm
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
Commit message: Ver 5
Parts:
- removed MC2: ESP32, ASTRAfootprints:ESP32-WROOM-32D-Devkit
- added REF**: MountingHole_2.7mm, MountingHole:MountingHole_2.7mm, F.Cu at (341.4, -71.4)
- added REF**: MountingHole_2.7mm, MountingHole:MountingHole_2.7mm, F.Cu at (93.5, 91.5)
- added REF**: MountingHole_2.7mm, MountingHole:MountingHole_2.7mm, F.Cu at (287.1, -40.5)
- added REF**: MountingHole_2.7mm, MountingHole:MountingHole_2.7mm, F.Cu at (151.5, 91.5)
- added REF**: MountingHole_2.7mm, MountingHole:MountingHole_2.7mm, F.Cu at (287.1, -71.4)
- added REF**: PinHeader_2x20_P2.54mm_Vertical, Connector_PinHeader_2.54mm:PinHeader_2x20_P2.54mm_Vertical, F.Cu at (98.3, 92.9)
- added REF**: MountingHole_2.7mm, MountingHole:MountingHole_2.7mm, F.Cu at (341.4, -40.5)
- added REF**: MountingHole_2.7mm, MountingHole:MountingHole_2.7mm, F.Cu at (93.5, 114.5)
- added U2: ESP32-WROOM-32E, RF_Module:ESP32-WROOM-32E, F.Cu at (165.5, 82.3)
- B1: footprint Connector_PinSocket_2.54mm:PinSocket_1x04_P2.54mm_Vertical -> TerminalBlock:TerminalBlock_MaiXu_MX126-5.0-04P_1x04_P5.00mm
- P1: footprint Connector_PinSocket_2.54mm:PinSocket_1x03_P2.54mm_Vertical -> TerminalBlock:TerminalBlock_MaiXu_MX126-5.0-02P_1x02_P5.00mm
- SW1, SW2, SW3, SW4, SW5, SW6, SW7: footprint Connector_PinSocket_2.54mm:PinSocket_1x02_P2.54mm_Vertical -> TerminalBlock:TerminalBlock_MaiXu_MX126-5.0-02P_1x02_P5.00mm
- moved D1 90.9 mm to (112.8, 122.5), turned to 90 degrees
- moved C6 89.2 mm to (99.8, 108.7), turned to -90 degrees
- moved D2 88.9 mm to (116.8, 122.5), turned to 90 degrees
- moved D3 87.1 mm to (120.8, 122.5), turned to 90 degrees
- moved C1 86.4 mm to (93.3, 102.0)
- moved R1 86.3 mm to (114.8, 122.5), turned to -90 degrees
- moved D4 85.5 mm to (124.8, 122.5), turned to 90 degrees
- moved S1 85.2 mm to (92.2, 122.5)
- moved R2 84.5 mm to (118.8, 122.5), turned to -90 degrees
- moved D5 84.0 mm to (128.8, 122.5), turned to 90 degrees
- moved R3 82.9 mm to (122.8, 122.5), turned to -90 degrees
- moved R4 81.4 mm to (126.8, 122.5), turned to -90 degrees
- moved J3 81.1 mm to (103.2, 84.2), turned to 180 degrees
- moved R5 80.2 mm to (130.8, 122.5), turned to -90 degrees
- moved SW2 64.2 mm to (184.4, 120.3)
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Routing:
- net +3.3V: track 177.0 -> 0.00 mm
- net /SDA: track 107.7 -> 0.00 mm
- net /SCL: track 102.2 -> 0.00 mm
- net +5V: track 101.9 -> 0.00 mm
- net /T1_DIAG: track 52.6 -> 0.00 mm
- net +12V: track 46.9 -> 0.00 mm
- net /T2_DIAG: track 40.6 -> 0.00 mm
- net GND: track 31.6 -> 0.00 mm
- net /2UART: track 22.6 -> 0.00 mm
- net /RED: track 19.3 -> 0.00 mm
- net /BLUE: track 19.2 -> 0.00 mm
- net /2PDN: track 18.8 -> 0.00 mm
- net /2STEP: track 18.8 -> 0.00 mm
- net /GREEN: track 16.1 -> 0.00 mm
- net /YELLOW: track 14.9 -> 0.00 mm
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Other:
- board size 55 x 85 mm -> 85 x 55 mm

Commit message: ver 5
Parts:
- removed REF** (x7): MountingHole_2.7mm, MountingHole:MountingHole_2.7mm
- removed REF**: PinHeader_2x20_P2.54mm_Vertical, Connector_PinHeader_2.54mm:PinHeader_2x20_P2.54mm_Vertical
- added C10: 10nF, Capacitor_SMD:C_0805_2012Metric_Pad1.18x1.45mm_HandSolder, F.Cu at (-53.3, 78.2)
- added C8: 100nF, Capacitor_SMD:C_0805_2012Metric_Pad1.18x1.45mm_HandSolder, F.Cu at (-53.3, 72.1)
- added C9: 100nF, Capacitor_SMD:C_0805_2012Metric_Pad1.18x1.45mm_HandSolder, F.Cu at (-53.3, 75.2)
- added G1: BNO085, Connector_PinSocket_2.54mm:PinSocket_1x09_P2.54mm_Vertical, F.Cu at (-48.6, 54.9)
- added J4: RJ45 (BNO085), Connector_RJ:RJ45_Amphenol_54602-x08_Horizontal, F.Cu at (-79.5, 37.6)
- added R6: 10kR, Resistor_SMD:R_0805_2012Metric_Pad1.20x1.40mm_HandSolder, F.Cu at (-64.0, 49.0)
- added U3: CH340C, Package_SO:SOIC-16_3.9x9.9mm_P1.27mm, F.Cu at (-57.4, 38.7)
- added U4: SPX3819M5-L-3-3, Package_TO_SOT_SMD:SOT-23-5, F.Cu at (-93.7, 76.8)
- B1: footprint TerminalBlock:TerminalBlock_MaiXu_MX126-5.0-04P_1x04_P5.00mm -> ASTRAfootprints:Double 1x02 screw connector
- P1, SW1, SW2, SW3, SW4, SW5, SW6, SW7: footprint TerminalBlock:TerminalBlock_MaiXu_MX126-5.0-02P_1x02_P5.00mm -> TerminalBlock:TerminalBlock_Xinya_XY308-2.54-2P_1x02_P2.54mm_Horizontal
- S1: footprint Connector_PinSocket_2.54mm:PinSocket_1x08_P2.54mm_Vertical -> ASTRAfootprints:Quadruple 1x02 screw connector
- moved SW5 290.3 mm to (-85.0, 3.14)
- moved SW6 285.8 mm to (-77.4, 3.14)
- moved U2 285.0 mm to (-112.3, 18.7)
- moved SW2 283.6 mm to (-69.7, -5.67)
- moved J1 272.7 mm to (-132.5, 37.6), turned to 0 degrees
- moved J5 262.5 mm to (-81.7, 9.98), turned to 0 degrees
- moved SW1 252.9 mm to (-77.4, -5.67)
- moved SW3 243.9 mm to (-62.1, -5.67), turned to 0 degrees
- moved P1 242.1 mm to (-85.0, -5.67)
- moved J2 239.1 mm to (-114.9, 37.6), turned to 0 degrees
- moved D5 230.1 mm to (-98.6, 88.1), turned to 0 degrees
- moved SW4 229.4 mm to (-54.4, -5.67), turned to 0 degrees
- moved T1 228.1 mm to (-92.2, 63.5), turned to 0 degrees
- moved SW7 227.7 mm to (-69.7, 3.14)
- moved D4 226.6 mm to (-98.6, 85.1), turned to 0 degrees
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Connections:
- C7 pad 1: Net-(C7-Pad1) -> GND
- J5 pad 2: unconnected-(J5-D--Pad2) -> Net-(J5-D-)
- J5 pad 3: unconnected-(J5-D+-Pad3) -> Net-(J5-D+)
- SW7 pad 2: Net-(C7-Pad1) -> Net-(U2-EN)
- U2 pad 25: unconnected-(U2-IO0-Pad25) -> /DTR
- U2 pad 34: unconnected-(U2-RXD0/IO3-Pad34) -> /UART2
- U2 pad 35: unconnected-(U2-TXD0/IO1-Pad35) -> /UART1
Routing:
- net Net-(D5-A): track 2.02 -> 0.00 mm
- net Net-(D4-A): track 2.01 -> 0.00 mm
- net Net-(D3-A): track 2.01 -> 0.00 mm
- net Net-(D2-A): track 2.01 -> 0.00 mm
- net Net-(D1-A): track 2.01 -> 0.00 mm
Other:
- board outline removed

Commit message: ver with ESP32UE
Parts:
- removed G1: BNO085, Connector_PinSocket_2.54mm:PinSocket_1x09_P2.54mm_Vertical
- removed J4: RJ45 (BNO085), Connector_RJ:RJ45_Amphenol_54602-x08_Horizontal
- removed U2: ESP32-WROOM-32E, RF_Module:ESP32-WROOM-32E
- added C11: 100nF, Capacitor_SMD:C_0402_1005Metric, F.Cu at (148.6, 86.6)
- added C12: 100nF, Capacitor_SMD:C_0402_1005Metric, F.Cu at (161.6, 84.9)
- added C13: 100nF, Capacitor_SMD:C_0402_1005Metric, F.Cu at (166.4, 107.9)
- added C15: 10uF, Capacitor_SMD:C_0402_1005Metric, F.Cu at (101.3, 84.4)
- added C16: 100nF, Capacitor_SMD:C_0402_1005Metric, F.Cu at (101.3, 85.4)
- added C17: 47uF, Capacitor_SMD:C_1206_3216Metric, F.Cu at (164.1, 84.6)
- added C18: 1uF, Capacitor_SMD:C_0402_1005Metric, F.Cu at (166.4, 108.9)
- added R7: 4.7kR, Resistor_SMD:R_0402_1005Metric, F.Cu at (137.0, 102.0)
- added R8: 4.7kR, Resistor_SMD:R_0402_1005Metric, F.Cu at (137.0, 103.0)
- added REF**: MountingHole_2.5mm, MountingHole:MountingHole_2.5mm, F.Cu at (171.6, 111.7)
- added REF**: MountingHole_2.5mm, MountingHole:MountingHole_2.5mm, F.Cu at (171.6, 68.3)
- added REF**: MountingHole_2.5mm, MountingHole:MountingHole_2.5mm, F.Cu at (93.2, 68.3)
- added REF**: MountingHole_2.5mm, MountingHole:MountingHole_2.5mm, F.Cu at (93.2, 111.7)
- added U5: ESP32-WROOM-32UE, RF_Module:ESP32-WROOM-32UE, F.Cu at (157.4, 97.0)
- C10, C2, C3, C4, C5, C6, C7, C8, C9: footprint Capacitor_SMD:C_0805_2012Metric_Pad1.18x1.45mm_HandSolder -> Capacitor_SMD:C_0402_1005Metric
- D1, D2, D3, D4, D5: footprint LED_SMD:LED_0805_2012Metric_Pad1.15x1.40mm_HandSolder -> LED_SMD:LED_0805_2012Metric
- R1, R2, R3, R4, R5, R6: footprint Resistor_SMD:R_0805_2012Metric_Pad1.20x1.40mm_HandSolder -> Resistor_SMD:R_0402_1005Metric
- moved S1 290.0 mm to (188.1, 66.8), turned to 90 degrees
- moved J1 281.4 mm to (145.7, 79.6), turned to 180 degrees
- moved SW6 268.9 mm to (170.9, 106.3), turned to 90 degrees
- moved SW5 268.6 mm to (161.0, 111.0)
- moved J5 252.8 mm to (161.9, 77.4), turned to 180 degrees
- moved J2 247.8 mm to (129.3, 79.6), turned to 180 degrees
- moved SW1 241.7 mm to (134.3, 111.0)
- moved SW2 240.8 mm to (140.9, 111.0)
- moved SW3 240.0 mm to (147.6, 111.0)
- moved SW4 239.1 mm to (154.3, 111.0)
- moved SW7 235.8 mm to (143.9, 102.8), turned to -90 degrees
- moved T1 231.2 mm to (137.2, 92.8), turned to -90 degrees
- moved U3 217.7 mm to (155.9, 82.7), turned to -90 degrees
- moved C9 215.7 mm to (162.3, 80.0)
- moved R6 215.2 mm to (148.1, 85.1), turned to 90 degrees
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Routing:
- net +3.3V: track 0.00 -> 174.5 mm, vias 0 -> 1
- net +5V: track 0.00 -> 103.9 mm
- net /1EN: track 0.00 -> 94.7 mm, vias 0 -> 1
- net /SCL: track 0.00 -> 86.6 mm
- net /SDA: track 0.00 -> 80.9 mm, vias 0 -> 2
- net GND: track 0.00 -> 65.7 mm, vias 0 -> 5
- net /1STEP: track 0.00 -> 64.4 mm, vias 0 -> 1
- net /1DIR: track 0.00 -> 62.5 mm, vias 0 -> 1
- net +12V: track 0.00 -> 58.7 mm
- net /1PDN: track 0.00 -> 52.5 mm, vias 0 -> 1
- net /1UART: track 0.00 -> 52.0 mm, vias 0 -> 1
- net /BLUE: track 0.00 -> 50.8 mm
- net /RED: track 0.00 -> 44.9 mm, vias 0 -> 1
- net /RETURN: track 0.00 -> 43.7 mm
- net /YELLOW: track 0.00 -> 43.5 mm
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Other:
- board outline added: 85 x 50 mm
- board text added: "ASTRA V0.2"
- board text added: "Buck"
